Commit message: Manual robot control console

File: edo/urdf/edo.urdf.xacro (robot description, xacro)
@@ -5,4 +5,6 @@
     <!--Import the edo macro -->
     <xacro:include filename="$(find edo)/urdf/edo.xacro"/>
+    <!--Import the box macro -->
+    <xacro:include filename="$(find edo)/urdf/pick_box.xacro"/>
     <xacro:arg name="hardware_interface" default="hardware_interface/PositionJointInterface"/>
     <xacro:arg name="robot_name" default="edo"/>

File: edo/urdf/edo.xacro (robot description, xacro)
@@ -12,5 +12,7 @@
     <xacro:property name="max_velocity" value="1.5"/>
     <xacro:property name="robot_prefix" value="edo"/>
-    <xacro:property name="table_offset" value="0.05"/>
+    <xacro:property name="table_width" value="1.5"/> <!-- x -->
+    <xacro:property name="table_depth" value="1.5"/> <!-- y -->
+    <xacro:property name="table_height" value="0.05"/> <!-- z -->
     <xacro:macro name="edo" params="parent hardware_interface robot_name *origin">
         <!--joint between {parent} and table_link-->
@@ -22,16 +24,22 @@
         <link name="${robot_prefix}_table_link">
             <visual>
-                <origin xyz="0 0 0.05" rpy="0 0 0"/>
-                <geometry>
-                    <box size="1 1 ${table_offset}"/>
-                </geometry>
-            </visual>
-            <collision>
-                <origin xyz="0 0 0.05" rpy="0 0 0"/>
-                <geometry>
-                    <box size="1 1 ${table_offset}"/>
+                <origin xyz="0 0 ${table_height}" rpy="0 0 0"/>
+                <geometry>
+                    <box size="${table_width} ${table_depth} ${table_height}"/>
+                    <!--mesh filename="package://edo/meshes/visual/table.dae"/-->
+                </geometry>
+            </visual>
+            <collision>
+                <origin xyz="0 0 ${table_height}" rpy="0 0 0"/>
+                <geometry>
+                    <box size="${table_width} ${table_depth} ${table_height}"/>
                 </geometry>
                 <material name="Grey"/>
             </collision>
+            <inertial>
+                <origin xyz="0 0 ${table_height}" rpy="0 0 0"/>
+                <mass value="30.0" />
+                <inertia  ixx="5.63125" ixy="11.25"  ixz="0"  iyy="0"  iyz="0"  izz="5.63125" />
+            </inertial>
         </link>
         <!--joint between table_link and base_link-->
@@ -39,5 +47,5 @@
             <parent link="${robot_prefix}_table_link"/>
             <child link="${robot_prefix}_base_link"/>
-            <origin xyz="0 0 ${table_offset}" rpy="0 0 0"/>
+            <origin xyz="0 0 ${table_height + 0.025}" rpy="0 0 0"/>
         </joint>
         <link name="${robot_prefix}_base_link">

Commit message: Fix last commit, pick n place trajectory

File: edo/urdf/edo.urdf.xacro (robot description, xacro)
@@ -5,6 +5,4 @@
     <!--Import the edo macro -->
     <xacro:include filename="$(find edo)/urdf/edo.xacro"/>
-    <!--Import the box macro -->
-    <xacro:include filename="$(find edo)/urdf/pick_box.xacro"/>
     <xacro:arg name="hardware_interface" default="hardware_interface/PositionJointInterface"/>
     <xacro:arg name="robot_name" default="edo"/>

File: edo/urdf/edo.xacro (robot description, xacro)
@@ -29,4 +29,5 @@
                     <!--mesh filename="package://edo/meshes/visual/table.dae"/-->
                 </geometry>
+                <material name="Grey"/>
             </visual>
             <collision>
@@ -35,5 +36,4 @@
                     <box size="${table_width} ${table_depth} ${table_height}"/>
                 </geometry>
-                <material name="Grey"/>
             </collision>
             <inertial>
@@ -41,4 +41,29 @@
                 <mass value="30.0" />
                 <inertia  ixx="5.63125" ixy="11.25"  ixz="0"  iyy="0"  iyz="0"  izz="5.63125" />
+            </inertial>
+        </link>
+        <!--joint between table_link and cartesian_target_link-->
+        <joint name="$${robot_name}_joint_c" type="fixed">
+            <parent link="${robot_prefix}_table_link"/>
+            <child link="${robot_prefix}_cartesian_target"/>
+        </joint>
+        <link name="${robot_prefix}_cartesian_target">
+            <visual>
+                <origin xyz="0 0.5 0.1" rpy="0 0 0"/>
+                <geometry>
+                    <box size="${table_width / 4} 0.05 0.05"/>
+                </geometry>
+                <material name="Blue"/>
+            </visual>
+            <collision>
+                <origin xyz="0 0.5 0.1" rpy="0 0 0"/>
+                <geometry>
+                    <box size="${table_width / 4} 0.05 0.05"/>
+                </geometry>
+            </collision>
+            <inertial>
+                <origin xyz="0 0.5 0.1" rpy="0 0 0"/>
+                <mass value="1.0" />
+                <inertia  ixx="0" ixy="0"  ixz="0"  iyy="0"  iyz="0"  izz="0" />
             </inertial>
         </link>

File: edo/urdf/edo_gripper_dummy.xacro (robot description, xacro)
@@ -201,10 +201,10 @@
                     <gripper_link>${robot_prefix}_gripper_right_finger_link</gripper_link>
                 </arm>
-                <forces_angle_tolerance>0</forces_angle_tolerance>
+                <forces_angle_tolerance>90</forces_angle_tolerance>
                 <update_rate>16</update_rate>
-                <grip_count_threshold>2</grip_count_threshold>
-                <max_grip_count>3</max_grip_count>
-                <release_tolerance>0.0005</release_tolerance>
-                <disable_collisions_on_attach>false</disable_collisions_on_attach>
+                <grip_count_threshold>1</grip_count_threshold>
+                <max_grip_count>8</max_grip_count>
+                <release_tolerance>0.005</release_tolerance>
+                <disable_collisions_on_attach>true</disable_collisions_on_attach>
                 <contact_topic>__default_topic__</contact_topic>
             </plugin>
