Commit message: Added test table

File: edo/urdf/edo.xacro (robot description, xacro)
@@ -12,10 +12,32 @@
     <xacro:property name="max_velocity" value="1.5"/>
     <xacro:property name="robot_prefix" value="edo"/>
+    <xacro:property name="table_offset" value="0.05"/>
     <xacro:macro name="edo" params="parent hardware_interface robot_name *origin">
-        <!--joint between {parent} and base_link-->
+        <!--joint between {parent} and table_link-->
         <joint name="${parent}_${robot_name}_joint" type="fixed">
             <xacro:insert_block name="origin"/>
             <parent link="${parent}"/>
+            <child link="${robot_prefix}_table_link"/>
+        </joint>
+        <link name="${robot_prefix}_table_link">
+            <visual>
+                <origin xyz="0 0 0.05" rpy="0 0 0"/>
+                <geometry>
+                    <box size="1 1 ${table_offset}"/>
+                </geometry>
+            </visual>
+            <collision>
+                <origin xyz="0 0 0.05" rpy="0 0 0"/>
+                <geometry>
+                    <box size="1 1 ${table_offset}"/>
+                </geometry>
+                <material name="Grey"/>
+            </collision>
+        </link>
+        <!--joint between table_link and base_link-->
+        <joint name="${robot_name}_joint0" type="fixed">
+            <parent link="${robot_prefix}_table_link"/>
             <child link="${robot_prefix}_base_link"/>
+            <origin xyz="0 0 ${table_offset}" rpy="0 0 0"/>
         </joint>
         <link name="${robot_prefix}_base_link">

Commit message: XYZ-RPY traj computation, better console commands

File: edo/urdf/edo.xacro (robot description, xacro)
@@ -12,7 +12,7 @@
     <xacro:property name="max_velocity" value="1.5"/>
     <xacro:property name="robot_prefix" value="edo"/>
-    <xacro:property name="table_width" value="1.5"/> <!-- x -->
-    <xacro:property name="table_depth" value="1.5"/> <!-- y -->
-    <xacro:property name="table_height" value="0.05"/> <!-- z -->
+    <xacro:property name="table_width" value="6.0"/> <!-- x -->
+    <xacro:property name="table_depth" value="4.0"/> <!-- y -->
+    <xacro:property name="table_height" value="1.6173"/> <!-- z -->
     <xacro:macro name="edo" params="parent hardware_interface robot_name *origin">
         <!--joint between {parent} and table_link-->
@@ -24,46 +24,19 @@
         <link name="${robot_prefix}_table_link">
             <visual>
-                <origin xyz="0 0 ${table_height}" rpy="0 0 0"/>
+                <origin xyz="0 0 0" rpy="0 0 0"/>
+                <geometry>
+                    <mesh filename="package://edo/meshes/visual/table.dae" scale="0.75 0.75 1"/>
+                </geometry>
+            </visual>
+            <collision>
+                <origin xyz="0 0 ${table_height / 2}" rpy="0 0 0"/>
                 <geometry>
                     <box size="${table_width} ${table_depth} ${table_height}"/>
-                    <!--mesh filename="package://edo/meshes/visual/table.dae"/-->
-                </geometry>
-                <material name="Grey"/>
-            </visual>
-            <collision>
-                <origin xyz="0 0 ${table_height}" rpy="0 0 0"/>
-                <geometry>
-                    <box size="${table_width} ${table_depth} ${table_height}"/>
-                </geometry>
-            </collision>
-            <inertial>
-                <origin xyz="0 0 ${table_height}" rpy="0 0 0"/>
+                </geometry>
+            </collision>
+            <inertial>
+                <origin xyz="0 0 ${table_height / 2}" rpy="0 0 0"/>
                 <mass value="30.0" />
-                <inertia  ixx="5.63125" ixy="11.25"  ixz="0"  iyy="0"  iyz="0"  izz="5.63125" />
-            </inertial>
-        </link>
-        <!--joint between table_link and cartesian_target_link-->
-        <joint name="$${robot_name}_joint_c" type="fixed">
-            <parent link="${robot_prefix}_table_link"/>
-            <child link="${robot_prefix}_cartesian_target"/>
-        </joint>
-        <link name="${robot_prefix}_cartesian_target">
-            <visual>
-                <origin xyz="0 0.5 0.1" rpy="0 0 0"/>
-                <geometry>
-                    <box size="${table_width / 4} 0.05 0.05"/>
-                </geometry>
-                <material name="Blue"/>
-            </visual>
-            <collision>
-                <origin xyz="0 0.5 0.1" rpy="0 0 0"/>
-                <geometry>
-                    <box size="${table_width / 4} 0.05 0.05"/>
-                </geometry>
-            </collision>
-            <inertial>
-                <origin xyz="0 0.5 0.1" rpy="0 0 0"/>
-                <mass value="1.0" />
-                <inertia  ixx="0" ixy="0"  ixz="0"  iyy="0"  iyz="0"  izz="0" />
+                <inertia  ixx="11.25" ixy="0"  ixz="0"  iyy="11.25"  iyz="0"  izz="11.25" />
             </inertial>
         </link>
@@ -72,5 +45,5 @@
             <parent link="${robot_prefix}_table_link"/>
             <child link="${robot_prefix}_base_link"/>
-            <origin xyz="0 0 ${table_height + 0.025}" rpy="0 0 0"/>
+            <origin xyz="0 0 ${table_height}" rpy="0 0 0"/>
         </joint>
         <link name="${robot_prefix}_base_link">

Commit message: Joint control GUI

File: edo/urdf/edo.xacro (robot description, xacro)
@@ -12,7 +12,7 @@
     <xacro:property name="max_velocity" value="1.5"/>
     <xacro:property name="robot_prefix" value="edo"/>
-    <xacro:property name="table_width" value="6.0"/> <!-- x -->
-    <xacro:property name="table_depth" value="4.0"/> <!-- y -->
-    <xacro:property name="table_height" value="1.6173"/> <!-- z -->
+    <xacro:property name="table_width" value="1.29657"/> <!-- x -->
+    <xacro:property name="table_depth" value="1.29657"/> <!-- y -->
+    <xacro:property name="table_height" value="0.83"/> <!-- z -->
     <xacro:macro name="edo" params="parent hardware_interface robot_name *origin">
         <!--joint between {parent} and table_link-->
@@ -26,9 +26,9 @@
                 <origin xyz="0 0 0" rpy="0 0 0"/>
                 <geometry>
-                    <mesh filename="package://edo/meshes/visual/table.dae" scale="0.75 0.75 1"/>
-                </geometry>
-            </visual>
-            <collision>
-                <origin xyz="0 0 ${table_height / 2}" rpy="0 0 0"/>
+                    <mesh filename="package://edo/meshes/visual/table.dae" scale="0.897 0.897 1"/>
+                </geometry>
+            </visual>
+            <collision>
+                <origin xyz="0 0 ${table_height / 2}" rpy="0 0 ${1.57 / 2}"/>
                 <geometry>
                     <box size="${table_width} ${table_depth} ${table_height}"/>
@@ -36,5 +36,5 @@
             </collision>
             <inertial>
-                <origin xyz="0 0 ${table_height / 2}" rpy="0 0 0"/>
+                <origin xyz="0 0 ${table_height / 2}" rpy="0 0 ${1.57 / 2}"/>
                 <mass value="30.0" />
                 <inertia  ixx="11.25" ixy="0"  ixz="0"  iyy="11.25"  iyz="0"  izz="11.25" />
@@ -62,5 +62,5 @@
                 <origin xyz="0 0 0.135" rpy="0 0 0"/>
                 <geometry>
-                    <mesh filename="package://edo/meshes/visual/link_0.dae"/>
+                    <mesh filename="package://edo/meshes/visual/off_center_link_0.dae"/>
                 </geometry>
             </visual>
@@ -68,5 +68,5 @@
                 <origin xyz="0 0 0.135" rpy="0 0 0"/>
                 <geometry>
-                    <mesh filename="package://edo/meshes/collision/link_0.dae"/>
+                    <mesh filename="package://edo/meshes/collision/off_center_link_0.dae"/>
                 </geometry>
                 <material name="Grey"/>
