Commit message: IKFast inverse kinematics implementation, EdoConsole class, minor bugfixes

File: edo/urdf/cylinder.urdf (robot description, URDF)
Before this commit: robot cilinder, 1 links, 0 joints
Links:
- removed link cilinder
- added link cylinder, mass 1.0; collision mesh filename=package://edo/meshes/visual/cylinder.dae scale=0.04 0.04 0.1; visual mesh filename=package://edo/meshes/visual/cylinder.dae scale=0.04 0.04 0.1

File: edo/urdf/edo_gripper_dummy.xacro (robot description, xacro)
@@ -202,5 +202,5 @@
                 </arm>
                 <forces_angle_tolerance>90</forces_angle_tolerance>
-                <update_rate>16</update_rate>
+                <update_rate>32</update_rate>
                 <grip_count_threshold>1</grip_count_threshold>
                 <max_grip_count>2</max_grip_count>

Commit message: Fixed pick and place by modifying cylinder spawning

File: edo/urdf/cylinder.urdf (robot description, URDF)
Before this commit: robot cylinder, 1 links, 0 joints
Links:
- link cylinder: geometry collision mesh filename=package://edo/meshes/visual/cylinder.dae; visual mesh filename=package://edo/meshes/visual/cylinder.dae
